File: 1. PCB/gps_tracer.kicad_sch (KiCad schematic)
At the start: 88 parts, among them IC1 TC4056A, J1 Mic, J2 SPK, J3 I2C, J4 BATTERY, J5 Micro_SD_Card, P1 USB_C_Plug_USB2.0, Q1 S8050, Q2 S8050, Q3 FDN358P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

Commit message: SIM800l receive and send sms, and answer on call my number
Other:
- note removed: "Додатифутпрінт на дросель"
- note removed: "Які значення резисторів дільників напруги?"
Changed lines of the file:
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@@
     (effects (font (size 1.27 1.27) (thickness 0.254) bold) (justify left bottom))
-  )
-  (text "Додатифутпрінт на дросель" (at 513.08 474.98 0)
-    (effects (font (size 3 3) bold) (justify left bottom))
   )
   (text "GSM" (at 756.92 128.27 0)
@@
     (effects (font (size 1.27 1.27) bold) (justify left bottom))
   )
-  (text "Які значення резисторів дільників напруги?\n" (at 556.26 528.32 0)
-    (effects (font (size 3 3) bold) (justify left bottom))
-  )
   (text "Vout (Must be 4.1 V)" (at 596.9 477.52 0)
