File: 1. PCB 3.1 version/gps_tracer.kicad_sch (KiCad schematic)
At the start: 98 parts, among them IC1 TC4056A, J1 Mic, J2 SPK, J3 I2C, J4 BATTERY, J5 Micro_SD_Card, P1 USB_C_Plug_USB2.0, Q1 S8050, Q2 S8050, Q3 FDN358P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

Commit message: finiched work with GPS loging into file
Parts:
- removed SW1: EN, Button_Switch_SMD:SW_Push_SPST_NO_Alps_SKRK, symbol Switch:SW_Push
- removed SW2: BOOT, Button_Switch_SMD:SW_Push_SPST_NO_Alps_SKRK, symbol Switch:SW_Push
- added JP7: EN, Resistor_SMD:R_0603_1608Metric_Pad0.98x0.95mm_HandSolder, symbol Jumper:Jumper_2_Open
- added JP7: BOOT, Resistor_SMD:R_0603_1608Metric_Pad0.98x0.95mm_HandSolder, symbol Jumper:Jumper_2_Open
Connections:
- net GND: now also JP7.1 (A), JP7.2 (B)
- net at C6.1, R12.1: now also JP7.1 (A)
- net at C6.1, R12.2, R12.2: now also JP7.2 (B)
Changed lines of the file:
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@@
     )
   )
+  (symbol (lib_id "Jumper:Jumper_2_Open") (at 241.3 71.12 0) (unit 1)
+    (in_bom yes) (on_board yes) (dnp no)
+    (property "Reference" "JP7" (at 241.3 63.5 0)
+      (effects (font (size 1.27 1.27)))
+    )
+    (property "Value" "EN" (at 241.3 67.31 0)
+      (effects (font (size 1.27 1.27)))
+    )
+    (property "Footprint" "Resistor_SMD:R_0603_1608Metric_Pad0.98x0.95mm_HandSolder" (at 241.3 71.12 0)
+      (effects (font (size 1.27 1.27)) hide)
+    )
+    (property "Datasheet" "~" (at 241.3 71.12 0)
+      (effects (font (size 1.27 1.27)) hide)
+    )
+    (pin "1")
+    (pin "2")
+    (instances
+      (project "STM32_NRF24L01_Sleep_mode"
+        (path "/5f3d2b28-6618-42e3-8f6e-5239c06ad0be"
+          (reference "JP7") (unit 1)
+        )
+      )
+      (project "gps_tracer"
+        (path "/9d7eac0e-bf1e-4bf0-8888-7adcd8c24b95"
+          (reference "JP5") (unit 1)
+        )
+      )
+    )
+  )
   (symbol (lib_id "Device:R") (at 715.01 161.29 0) (mirror x) (unit 1)
     (in_bom yes) (on_board yes) (dnp no)
@@
     )
   )
-  (symbol (lib_id "Switch:SW_Push") (at 241.3 71.12 0) (unit 1)
-    (in_bom yes) (on_board yes) (dnp no) (fields_autoplaced)
-    (property "Reference" "SW1" (at 241.3 64.77 0)
-      (effects (font (size 1.27 1.27)))
-    )
-    (property "Value" "EN" (at 241.3 67.31 0)
-      (effects (font (size 1.27 1.27)))
-    )
-    (property "Footprint" "Button_Switch_SMD:SW_Push_SPST_NO_Alps_SKRK" (at 241.3 66.04 0)
-      (effects (font (size 1.27 1.27)) hide)
-    )
-    (property "Datasheet" "~" (at 241.3 66.04 0)
-      (effects (font (size 1.27 1.27)) hide)
-    )
-    (pin "1")
-    (pin "2")
-    (instances
-      (project "gps_tracer"
-        (path "/9d7eac0e-bf1e-4bf0-8888-7adcd8c24b95"
-          (reference "SW1") (unit 1)
-        )
-      )
-      (project "PCB"
-        (path "/f0559356-5a76-4eab-b33c-c712023883fc"
-          (reference "SW1") (unit 1)
-        )
-      )
-    )
-  )
   (symbol (lib_name "GND_2") (lib_id "power:GND") (at 137.795 410.845 0) (unit 1)
     (in_bom yes) (on_board yes) (dnp no)
@@
     )
   )
-  (symbol (lib_id "Switch:SW_Push") (at 341.63 71.12 0) (unit 1)
-    (in_bom yes) (on_board yes) (dnp no) (fields_autoplaced)
-    (property "Reference" "SW2" (at 341.63 64.77 0)
-      (effects (font (size 1.27 1.27)))
-    )
-    (property "Value" "BOOT" (at 341.63 67.31 0)
-      (effects (font (size 1.27 1.27)))
-    )
-    (property "Footprint" "Button_Switch_SMD:SW_Push_SPST_NO_Alps_SKRK" (at 341.63 66.04 0)
-      (effects (font (size 1.27 1.27)) hide)
-    )
-    (property "Datasheet" "~" (at 341.63 66.04 0)
-      (effects (font (size 1.27 1.27)) hide)
-    )
-    (pin "1")
-    (pin "2")
-    (instances
-      (project "gps_tracer"
-        (path "/9d7eac0e-bf1e-4bf0-8888-7adcd8c24b95"
-          (reference "SW2") (unit 1)
-        )
-      )
-      (project "PCB"
-        (path "/f0559356-5a76-4eab-b33c-c712023883fc"
-          (reference "SW2") (unit 1)
-        )
-      )
-    )
-  )
   (symbol (lib_id "Jumper:Jumper_2_Open") (at 59.055 389.255 0) (unit 1)
     (in_bom yes) (on_board yes) (dnp no)
@@
         )
       )
+    )
+  )
+  (symbol (lib_id "Jumper:Jumper_2_Open") (at 341.63 71.12 0) (unit 1)
+    (in_bom yes) (on_board yes) (dnp no)
+    (property "Reference" "JP7" (at 341.63 63.5 0)
+      (effects (font (size 1.27 1.27)))
+    )
+    (property "Value" "BOOT" (at 341.63 67.31 0)
+      (effects (font (size 1.27 1.27)))
+    )
+    (property "Footprint" "Resistor_SMD:R_0603_1608Metric_Pad0.98x0.95mm_HandSolder" (at 341.63 71.12 0)
+      (effects (font (size 1.27 1.27)) hide)
+    )
+    (property "Datasheet" "~" (at 341.63 71.12 0)
+      (effects (font (size 1.27 1.27)) hide)
+    )
+    (pin "1")
+    (pin "2")
+    (instances
+      (project "STM32_NRF24L01_Sleep_mode"
+        (path "/5f3d2b28-6618-42e3-8f6e-5239c06ad0be"
+          (reference "JP7") (unit 1)
+        )
+      )
+      (project "gps_tracer"
+        (path "/9d7eac0e-bf1e-4bf0-8888-7adcd8c24b95"
+          (reference "JP6") (unit 1)
+        )
+      )

Commit message: SIM800l receive and send sms, and answer on call my number
Parts:
- removed C6: 22u, Capacitor_SMD:C_0805_2012Metric_Pad1.18x1.45mm_HandSolder, symbol Device:C
- removed D1: BAT48ZFILM, Diode_SMD:D_SOD-123, symbol Diode:1N5819WS
- removed Q4: LTC4412, Package_TO_SOT_SMD:SOT-23, symbol Transistor_FET:IRLML6402
- removed R15: 470k, Resistor_SMD:R_0603_1608Metric_Pad0.98x0.95mm_HandSolder, symbol Device:R
- removed U10: LTC4412xS6, Package_TO_SOT_SMD:TSOT-23-6, symbol Power_Management:LTC4412xS6
Connections:
- net at C6.1, L1.1, U11.3 (Vcc)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: now also C6.1, C6.1, IC1.5 (BAT), J4.2 (Pin_2), R15.1, R15.1
Other:
- note added: "SS14"
- note added: "ПОМНІЯТИ ДІОД НА SS14 !!!"
- note removed: "5 Volt FROM USB"
- note removed: "Power source switcher"
- note removed: "Додатифутпрінт на дросель"
- note removed: "ПЕРЕВІРИТИ СХЕМУ"
- note removed: "Поміняти Футпрінт конденсатора на більший"
- note removed: "Які значення резисторів дільників напруги?"

Commit message: HTTP file server added into /Parts project/6. Web server/13. HTTP file server. The files in Micro SD card can be deleted or download from browser
Parts:
- removed J2: SPK, Footprint_library:JST 1.25, symbol Connector:Conn_01x02_Pin
- removed JP7: EN, Resistor_SMD:R_0603_1608Metric_Pad0.98x0.95mm_HandSolder, symbol Jumper:Jumper_2_Open
- added D1: GREEN LED, LED_SMD:LED_0603_1608Metric_Pad1.05x0.95mm_HandSolder, symbol Device:LED
- added D2: BLUE LED, LED_SMD:LED_0603_1608Metric_Pad1.05x0.95mm_HandSolder, symbol Device:LED
- added D4: YELLOW_LED, LED_SMD:LED_0603_1608Metric_Pad1.05x0.95mm_HandSolder, symbol Device:LED
- added R1, R15, R19: 700, Resistor_SMD:R_0603_1608Metric_Pad0.98x0.95mm_HandSolder, symbol Device:R
- added U10: PCA9536D, Package_SO:SOIC-8_3.9x4.9mm_P1.27mm, symbol Interface_Expansion:PCA9536D
- D5: value BAT48ZFILM -> SS14; footprint Diode_SMD:D_SOD-123 -> Diode_SMD:D_SMA
- D9: value LED -> RED LED
Connections:
- net +3.3V: now also U10.8 (VDD)
- net EXTERNAL_WOKE_UP: now also U4.26 (IO4)
- net GND: now also C6.1, R12.2, R12.2, D1.1 (K), D2.1 (K), D4.1 (K), U10.4 (VSS)
- net SCL: now also J3.1 (Pin_1), U10.6 (SCL); no longer J3.2 (Pin_2)
- net SDA: now also J3.2 (Pin_2), U10.7 (SDA); no longer J3.1 (Pin_1)
- net RED_LED: no longer names the net of R23.1
- net RED_LED: now also U10.1 (IO0); no longer U4.30 (IO18)
- new net: R1.1, U10.2 (IO1)
- new net: R15.1, U10.3 (IO2)
- new net: R19.1, U10.5 (IO3)
- new net: D2.2 (A), R15.2
- new net: D4.2 (A), R19.2
- new net: D1.2 (A), R1.2
- no-connect marks 39 -> 46
Other:
- note removed: "SS14"
- moved on the sheet: D9, J3, R23
